File: schematic/epromemu.kicad_sch (KiCad schematic)
At the start: 19 parts, among them J3 EPROM Connector, U1 Teensy4.1, U2 74HC245, U3 74HC245, U4 74HC245, U5 74HC245, U6 74HC32

Commit message: REV D
Parts:
- removed JP1: PWR, Connector_PinHeader_2.54mm:PinHeader_1x02_P2.54mm_Vertical, symbol Jumper:Jumper_2_Open
- JP1: renamed from JP2; footprint Connector_PinHeader_2.54mm:PinHeader_1x03_P2.54mm_Vertical -> MyFootprints:Jumper_1x03_P2.54mm_Vertical
- JP2: renamed from JP3; footprint Connector_PinHeader_2.54mm:PinHeader_1x03_P2.54mm_Vertical -> MyFootprints:Jumper_1x03_P2.54mm_Vertical
Connections:
- net JP1_PWR is gone; now on net +5V: J3.32 (Pin_32), JP1.1 (A), JP2.1 (A)
- net GND: now also U1.34 (GND), U1.47 (GND), U4.6 (A4), U4.7 (A5), U4.8 (A6), U4.9 (A7)
- no-connect marks 47 -> 41
Other:
- moved on the sheet: C2, C3, C4, C5, C6, H1, H2, H3, H4, J3, JP1, JP2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

Commit message: REV E (unproduced)
Parts:
- removed JP1: A17, MyFootprints:Jumper_1x03_P2.54mm_Vertical, symbol Jumper:Jumper_3_Open
- removed JP2: A13, MyFootprints:Jumper_1x03_P2.54mm_Vertical, symbol Jumper:Jumper_3_Open
- removed U6: 74HC32, Package_DIP:DIP-14_W7.62mm_Socket, symbol 74xx:74LS32
- added U5: SN74LVC1G32DBVR, Package_TO_SOT_SMD:SOT-23-5, symbol MySymbols:SN74LVC1G32DBVR
- C5: renamed from C6; footprint Capacitor_THT:C_Disc_D5.0mm_W2.5mm_P5.00mm -> Capacitor_SMD:C_0603_1608Metric_Pad1.08x0.95mm_HandSolder
- H1, H2, H3, H4: footprint MountingHole:MountingHole_2.2mm_M2_ISO7380_Pad -> MountingHole:MountingHole_2.2mm_M2_ISO7380
- U1: renamed from U5; value 74HC245 -> SN74LVC245AN; symbol 74xx:74HC245 -> MySymbols:SN74LVC245AN
- U2: renamed from U4; value 74HC245 -> SN74LVC245AN; symbol 74xx:74HC245 -> MySymbols:SN74LVC245AN
- U3: value 74HC245 -> SN74LVC245AN; symbol 74xx:74HC245 -> MySymbols:SN74LVC245AN
- U4: renamed from U2; value 74HC245 -> SN74LVC245AN; symbol 74xx:74HC245 -> MySymbols:SN74LVC245AN
- renumbered C5 to C1, C4 to C2, C2 to C4, J3 to J1, U1 to U6
Connections:
- net +3V3: now also C4.1, C5.1, U3.1 (A->B), U4.20 (VCC), U6.46 (3V3), U5.5 (VCC)
- net A0_3V3: now also U2.18 (B0); no longer U2.15 (B3)
- net A0_5V: now also U2.2 (A0); no longer U2.5 (A3)
- net A10_3V3: now also U3.18 (B0); no longer U3.9 (A7)
- net A10_5V: now also U3.2 (A0); no longer U3.11 (B7)
- net A11_3V3: now also U3.17 (B1); no longer U3.8 (A6)
- net A11_5V: now also U3.3 (A1); no longer U3.12 (B6)
- net A12_3V3: now also U1.14 (B4); no longer U1.15 (B3)
- net A12_5V: now also U1.6 (A4); no longer U1.5 (A3)
- net A13_3V3: now also U3.14 (B4); no longer U3.5 (A3)
- net A13_5V: now also J1.28 (Pin_28), U3.6 (A4); no longer U3.15 (B3)
- net A14_3V3: now also U3.13 (B5); no longer U3.4 (A2)
- net A14_5V: now also U3.7 (A5); no longer U3.16 (B2)
- net A15_3V3: now also U1.13 (B5); no longer U1.16 (B2)
- net A15_5V: now also U1.7 (A5); no longer U1.4 (A2)
- net A16_3V3: now also U1.12 (B6); no longer U1.17 (B1)
- net A16_5V: now also U1.8 (A6); no longer U1.3 (A1)
- net A17_3V3: now also U3.12 (B6); no longer U3.3 (A1)
- net A17_5V: now also J1.30 (Pin_30), U3.8 (A6); no longer U3.17 (B1)
- net A18_3V3: now also U3.11 (B7); no longer U3.2 (A0)
- net A18_5V: now also U3.9 (A7); no longer U3.18 (B0)
- net A19_3V3: now also U1.11 (B7); no longer U1.18 (B0)
- net A19_5V: now also U1.9 (A7); no longer U1.2 (A0)
- net A1_3V3: now also U2.17 (B1); no longer U2.16 (B2)
- net A1_5V: now also U2.3 (A1); no longer U2.4 (A2)
- net A2_3V3: now also U2.16 (B2); no longer U2.17 (B1)
- net A2_5V: now also U2.4 (A2); no longer U2.3 (A1)
- net A3_3V3: now also U2.15 (B3); no longer U2.18 (B0)
- net A3_5V: now also U2.5 (A3); no longer U2.2 (A0)
- net A4_3V3: now also U1.18 (B0); no longer U1.11 (B7)
- net A4_5V: now also U1.2 (A0); no longer U1.9 (A7)
- net A5_3V3: now also U1.17 (B1); no longer U1.12 (B6)
- net A5_5V: now also U1.3 (A1); no longer U1.8 (A6)
- net A6_3V3: now also U1.16 (B2); no longer U1.13 (B5)
- net A6_5V: now also U1.4 (A2); no longer U1.7 (A5)
- net A7_3V3: now also U1.15 (B3); no longer U1.14 (B4)
- net A7_5V: now also U1.5 (A3); no longer U1.6 (A4)
- net A8_3V3: now also U3.15 (B3); no longer U3.6 (A4)
- net A8_5V: now also U3.5 (A3); no longer U3.14 (B4)
- net A9_3V3: now also U3.16 (B2); no longer U3.7 (A5)
- net A9_5V: now also U3.4 (A2); no longer U3.13 (B5)
- net CE_5V: now also U5.2
- net D0_3V3: now also U4.13 (B5); no longer U4.4 (A2)
- net D0_5V: now also U4.7 (A5); no longer U4.16 (B2)
- net D1_3V3: now also U4.15 (B3); no longer U4.6 (A4)
- net D1_5V: now also U4.5 (A3); no longer U4.14 (B4)
- net D2_3V3: now also U4.17 (B1); no longer U4.8 (A6)
- net D2_5V: now also U4.3 (A1); no longer U4.12 (B6)
- net D3_3V3: now also U4.18 (B0); no longer U4.9 (A7)
- net D3_5V: now also U4.2 (A0); no longer U4.11 (B7)
- net D4_3V3: now also U4.16 (B2); no longer U4.7 (A5)
- net D4_5V: now also U4.4 (A2); no longer U4.13 (B5)
- net D5_3V3: now also U4.14 (B4); no longer U4.5 (A3)
- net D5_5V: now also U4.6 (A4); no longer U4.15 (B3)
- net D6_3V3: now also U4.12 (B6); no longer U4.3 (A1)
- net D6_5V: now also U4.8 (A6); no longer U4.17 (B1)
- net D7_3V3: now also U4.11 (B7); no longer U4.2 (A0)
- net D7_5V: now also U4.9 (A7); no longer U4.18 (B0)
- net GND: now also U4.1 (A->B), U5.3 (GND); no longer U3.1 (A->B)
- net OE_5V: now also U5.1
- net OE_CE: now reaches U4.19 (CE)
- net OE_CE: now also U5.4
- removed net +5V: C4.1, C5.1, J1.32 (Pin_32), U4.1 (A->B), U4.20 (VCC), U6.48 (VIN)
- no-connect marks 41 -> 20
Other:
- title: EPROM Emulator -> EPROMEmu
- moved on the sheet: C5, H1, H2, H3, H4

Commit message: REV F
Parts:
- removed C1: 0.1uf, Capacitor_THT:C_Disc_D5.0mm_W2.5mm_P5.00mm, symbol Device:C_Small
- removed C5: 0.1uf, Capacitor_SMD:C_0603_1608Metric_Pad1.08x0.95mm_HandSolder, symbol Device:C_Small
- removed U1, U2, U3, U4: SN74LVC245AN, Package_DIP:DIP-20_W7.62mm_Socket, symbol MySymbols:SN74LVC245AN
- removed U5: SN74LVC1G32DBVR, Package_TO_SOT_SMD:SOT-23-5, symbol MySymbols:SN74LVC1G32DBVR
- added U1, U2, U3: SN74LVC827APWR, Package_SO:SOIC-24W_7.5x15.4mm_P1.27mm, symbol MySymbols:SN74LVC827APWR
- C1: renamed from C3; footprint Capacitor_THT:C_Disc_D5.0mm_W2.5mm_P5.00mm -> Capacitor_SMD:C_0603_1608Metric_Pad1.08x0.95mm_HandSolder
- C2: footprint Capacitor_THT:C_Disc_D5.0mm_W2.5mm_P5.00mm -> Capacitor_SMD:C_0603_1608Metric_Pad1.08x0.95mm_HandSolder
- C3: renamed from C4; footprint Capacitor_THT:C_Disc_D5.0mm_W2.5mm_P5.00mm -> Capacitor_SMD:C_0603_1608Metric_Pad1.08x0.95mm_HandSolder
- renumbered U6 to U4
Connections:
- net +3V3: now also U1.24 (VCC), U2.24 (VCC), U3.24 (VCC); no longer U4.15 (3V3)
- net A0_3V3: now also U2.23 (Y1)
- net A0_5V: now also U2.2 (A1)
- net A10_3V3: now also U2.21 (Y3)
- net A10_5V: now also U2.4 (A3)
- net A11_3V3: now also U2.18 (Y6)
- net A11_5V: now also U2.7 (A6)
- net A12_3V3: now also U1.19 (Y5)
- net A12_5V: now also U1.6 (A5)
- net A13_3V3: now also U1.22 (Y2)
- net A13_5V: now also U1.3 (A2)
- net A14_3V3: now also U1.20 (Y4)
- net A14_5V: now also U1.5 (A4)
- net A15_3V3: now also U1.17 (Y7)
- net A15_5V: now also U1.8 (A7)
- net A16_3V3: now also U1.15 (Y9)
- net A16_5V: now also U1.10 (A9)
- net A17_3V3: now also U1.18 (Y6)
- net A17_5V: now also U1.7 (A6)
- net A18_3V3: now also U1.16 (Y8)
- net A18_5V: now also U1.9 (A8)
- net A19_3V3: now also U1.14 (Y1O)
- net A19_5V: now also U1.11 (A1O)
- net A1_3V3: now also U2.22 (Y2)
- net A1_5V: now also U2.3 (A2)
- net A2_3V3: now also U2.20 (Y4)
- net A2_5V: now also U2.5 (A4)
- net A3_3V3: now also U2.19 (Y5)
- net A3_5V: now also U2.6 (A5)
- net A4_3V3: now also U2.17 (Y7)
- net A4_5V: now also U2.8 (A7)
- net A5_3V3: now also U2.15 (Y9)
- net A5_5V: now also U2.10 (A9)
- net A6_3V3: now also U1.23 (Y1)
- net A6_5V: now also U1.2 (A1)
- net A7_3V3: now also U1.21 (Y3)
- net A7_5V: now also U1.4 (A3)
- net A8_3V3: now also U2.14 (Y1O)
- net A8_5V: now also U2.11 (A1O)
- net A9_3V3: now also U2.16 (Y8)
- net A9_5V: now also U2.9 (A8)
- net CE_5V: now also U3.13 (~{OE2})
- net D0_3V3: now also U3.4 (A3)
- net D0_5V: now also U3.21 (Y3)
- net D1_3V3: now also U3.6 (A5)
- net D1_5V: now also U3.19 (Y5)
- net D2_3V3: now also U3.8 (A7)
- net D2_5V: now also U3.17 (Y7)
- net D3_3V3: now also U3.9 (A8)
- net D3_5V: now also U3.16 (Y8)
- net D4_3V3: now also U3.7 (A6)
- net D4_5V: now also U3.18 (Y6)
- net D5_3V3: now also U3.5 (A4)
- net D5_5V: now also U3.20 (Y4)
- net D6_3V3: now also U3.3 (A2)
- net D6_5V: now also U3.22 (Y2)
- net D7_3V3: now also U3.2 (A1)
- net D7_5V: now also U3.23 (Y1)
- net GND: now also U1.1 (~{OE1}), U1.12 (GND), U1.13 (~{OE2}), U2.1 (~{OE1}), U2.12 (GND), U2.13 (~{OE2}), U3.10 (A9), U3.11 (A1O), U3.12 (GND)
- net OE_5V: now also U3.1 (~{OE1})
- no-connect marks 20 -> 19
Other:
- company: Brian Peek -> Ganksoft Entertainment
- moved on the sheet: C1, C3, J1, U4
